Commit message: Drake patch (#26)
* Adapt to namespace changes in pydrake.solvers

* Get mesh files from RobotLocomotion/models

File: models/j2s7s300_arm_sphere_collision.urdf (robot description, URDF)
Before this commit: robot j2s7s300_arm, 9 links, 8 joints
Links:
- link j2s7s300_link_1: geometry visual mesh filename=package://drake_models/jaco_description/meshes/ring_big.obj; visual mesh filename=package://drake_models/jaco_description/meshes/shoulder.obj
- link j2s7s300_link_2: geometry visual mesh filename=package://drake_models/jaco_description/meshes/arm_half_1.o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; visual mesh filename=package://drake_models/jaco_description/meshes/ring_big.obj
- link j2s7s300_link_3: geometry visual mesh filename=package://drake_models/jaco_description/meshes/arm_half_2.o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; visual mesh filename=package://drake_models/jaco_description/meshes/ring_big.obj
- link j2s7s300_link_4: geometry visual mesh filename=package://drake_models/jaco_description/meshes/forearm.obj; visual mesh filename=package://drake_models/jaco_description/meshes/ring_small.o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
- link j2s7s300_link_5: geometry visual mesh filename=package://drake_models/jaco_description/meshes/ring_small.o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; visual mesh filename=package://drake_models/jaco_description/meshes/wrist_spheri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
- link j2s7s300_link_6: geometry collision sphere radius=0.035; visual mesh filename=package://drake_models/jaco_description/meshes/ring_small.o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
- link j2s7s300_link_base: geometry visual mesh filename=package://drake_models/jaco_description/meshes/base.obj

File: models/j2s7s300_arm_sphere_collision_v2.urdf (robot description, URDF)
Before this commit: robot j2s7s300_arm, 9 links, 8 joints
Links:
- link j2s7s300_link_1: geometry collision sphere radius=0.045; visual mesh filename=package://drake_models/jaco_description/meshes/ring_big.obj
- link j2s7s300_link_2: geometry collision sphere radius=0.045; visual mesh filename=package://drake_models/jaco_description/meshes/arm_half_1.o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
- link j2s7s300_link_3: geometry collision sphere radius=0.025; collision sphere radius=0.045
- link j2s7s300_link_4: geometry collision sphere radius=0.025; collision sphere radius=0.045
- link j2s7s300_link_5: geometry collision sphere radius=0.035; visual mesh filename=package://drake_models/jaco_description/meshes/ring_small.o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
- link j2s7s300_link_6: geometry collision sphere radius=0.035; visual mesh filename=package://drake_models/jaco_description/meshes/ring_small.o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
- link j2s7s300_link_base: geometry visual mesh filename=package://drake_models/jaco_description/meshes/base.obj
